Commit message: "updated the effort controller with gazebo and a couple of launch files"

File: pendubot_description/pendubot/robot.urdf.xacro (robot description, xacro)
@@ -1,3 +1,5 @@
-<robot name="pendubot">
+<?xml version="1.0"?>
+<robot name="pendubot"  xmlns:xacro="http://wiki.ros.org/xacro">
+<xacro:include filename="$(find pendubot_description)/pendubot/ros2_control.urdf.xacro"/>
 <link name="support_plaform_1">
 <visual>
@@ -140,5 +142,5 @@
 </inertial>
 </link>
-<joint name="continuous_revolute 2" type="continuous">
+<joint name="continuous_revolute_2" type="continuous">
 <origin xyz="1.1102230246251565404e-16 -0.20000000000000006661 -0.025000000000000011796" rpy="3.141592653589793116 1.232595164407828209e-32 3.141592653589793116" />
 <parent link="cart_swinger" />
@@ -148,5 +150,5 @@
 <joint_properties friction="0.0"/>
 </joint>
-<joint name="continuous_revolute 1" type="continuous">
+<joint name="continuous_revolute_1" type="continuous">
 <origin xyz="0.10468245836551855199 0.024999999999999911182 0" rpy="-2.4651903288156618919e-32 -1.570796326794896336 0" />
 <parent link="cart_move" />
@@ -156,5 +158,5 @@
 <joint_properties friction="0.0"/>
 </joint>
-<joint name="slider 1" type="prismatic">
+<joint name="slider_1" type="prismatic">
 <origin xyz="-0.99499999999999999556 -0.025000000000000022204 -0.040000000000000021649" rpy="-0 -1.570796326794896558 0" />
 <parent link="cart_pole_line" />

Commit message: "I can start a branch here for where one balances with swinger one at the bottom and the other upright"

File: pendubot_description/pendubot/robot.urdf.xacro (robot description, xacro)
@@ -158,10 +158,10 @@
 <joint_properties friction="0.0"/>
 </joint>
-<joint name="slider_1" type="prismatic">
+<joint name="slider_1" type="fixed">
 <origin xyz="-0.99499999999999999556 -0.025000000000000022204 -0.040000000000000021649" rpy="-0 -1.570796326794896558 0" />
 <parent link="cart_pole_line" />
 <child link="cart_move" />
 <axis xyz="0 0 1"/>
-<limit effort="1" velocity="20" lower="-0.80000000000000004441" upper="0.80000000000000004441"/>
+<limit effort="1" velocity="20"/>
 <joint_properties friction="0.0"/>
 </joint>

File: pendubot_description/pendubot/ros2_control.urdf.xacro (robot description, xacro)
@@ -1,9 +1,9 @@
 <?xml version="1.0"?>
 <robot xmlns:xacro="http://www.ros.org/wiki/xacro">
-<ros2_control name="GazeboSimSystem" type="system">
+<ros2_control name="IgzSimSystem" type="system">
   <hardware>
-    <plugin>gazebo_ros2_control/GazeboSystem</plugin>
+    <plugin>ign_ros2_control/IgnitionSystem</plugin>
   </hardware>
-  <joint name="slider_1">
+  <!-- <joint name="slider_1">
     <command_interface name="position">
       <param name="min">-0.85</param>
@@ -15,5 +15,5 @@
     <state_interface name="velocity"/>
     <state_interface name="effort"/>
-  </joint>
+  </joint> -->
   <joint name="continuous_revolute_1">
     <command_interface name="effort">
@@ -33,8 +33,14 @@
   </joint>
 </ros2_control>
-  <gazebo>
+  <!-- <gazebo>
     <plugin filename="libgazebo_ros2_control.so" name="gazebo_ros2_control">
       <parameters>$(find pendubot_description)/config/effort_control.yaml</parameters>
     </plugin>
-  </gazebo>
+  </gazebo> -->
+<gazebo>
+    <plugin name="ign_ros2_control::IgnitionROS2ControlPlugin"
+        filename="ign_ros2_control-system">
+        <parameters>$(find pendubot_description)/config/effort_control.yaml</parameters>
+    </plugin>
+</gazebo>
 </robot>

Commit message: "Works in getting the pendubot to the top pendubot_description coming to add angular persuit"

File: pendubot_description/pendubot/robot.urdf.xacro (robot description, xacro)
@@ -20,5 +20,5 @@
 <inertial>
 <origin xyz="-0.084999999999999978351 0.0019366224157372038169 0.20527754982977566844" rpy="0 0 0"/>
-<mass value="8.3650792577619803581" />
+<mass value="800.3650792577619803581" />
 <inertia ixx="0.18809404056513884251" ixy="6.6429634534729561893e-19"  ixz="-3.3040840509945104842e-17" iyy="0.19768960892502629445" iyz="0.0034874963072423492694" izz="0.014632587595117504606" />
 </inertial>
@@ -64,5 +64,5 @@
 <inertial>
 <origin xyz="-0.018063377584262709646 -0.26472245017022433267 7.9318860187151341436e-17" rpy="0 0 0"/>
-<mass value="8.3650792577619803581" />
+<mass value="800.3650792577619803581" />
 <inertia ixx="0.19768960892502629445" ixy="0.0034874963072423744229"  ixz="2.639638845664999534e-49" iyy="0.014632587595117504606" iyz="2.3862418064830125439e-51" izz="0.18809404056513884251" />
 </inertial>
@@ -143,9 +143,10 @@
 </link>
 <joint name="continuous_revolute_2" type="continuous">
+<!-- <joint name="continuous_revolute_2" type="fixed"> -->
 <origin xyz="1.1102230246251565404e-16 -0.20000000000000006661 -0.025000000000000011796" rpy="3.141592653589793116 1.232595164407828209e-32 3.141592653589793116" />
 <parent link="cart_swinger" />
 <child link="cart_swinger_2" />
 <axis xyz="0 0 1"/>
-<limit effort="1" velocity="20" />
+<limit effort="10000" velocity="20" />
 <joint_properties friction="0.0"/>
 </joint>
@@ -155,5 +156,5 @@
 <child link="cart_swinger" />
 <axis xyz="0 0 1"/>
-<limit effort="1" velocity="20" />
+<limit effort="10000" velocity="20" />
 <joint_properties friction="0.0"/>
 </joint>

File: pendubot_description/pendubot/ros2_control.urdf.xacro (robot description, xacro)
@@ -1,24 +1,20 @@
 <?xml version="1.0"?>
 <robot xmlns:xacro="http://www.ros.org/wiki/xacro">
-<ros2_control name="IgzSimSystem" type="system">
-  <hardware>
-    <plugin>ign_ros2_control/IgnitionSystem</plugin>
-  </hardware>
-  <!-- <joint name="slider_1">
-    <command_interface name="position">
-      <param name="min">-0.85</param>
-      <param name="max">0.85</param>
-    </command_interface>
-    <state_interface name="position">
-      <param name="initial_value">0.0</param>
-    </state_interface>
-    <state_interface name="velocity"/>
-    <state_interface name="effort"/>
-  </joint> -->
-  <joint name="continuous_revolute_1">
-    <command_interface name="effort">
-      <param name="min">-1000</param>
-      <param name="max">1000</param>
-    </command_interface>
+  <ros2_control name="IgzSimSystem" type="system">
+    <hardware>
+      <plugin>ign_ros2_control/IgnitionSystem</plugin>
+    </hardware>
+    <joint name="continuous_revolute_1">
+      <command_interface name="effort">
+        <param name="min">-1000</param>
+        <param name="max">1000</param>
+      </command_interface>
+      <state_interface name="position">
+        <param name="initial_value">0.0</param>
+      </state_interface>
+      <state_interface name="velocity" />
+      <state_interface name="effort" />
+    </joint>
+    <joint name="continuous_revolute_2">
     <state_interface name="position">
        <param name="initial_value">0.0</param>
@@ -26,21 +22,10 @@
     <state_interface name="velocity"/>
   </joint>
-  <joint name="continuous_revolute_2">
-    <state_interface name="position">
-       <param name="initial_value">0.0</param>
-       </state_interface>
-    <state_interface name="velocity"/>
-  </joint>
-</ros2_control>
-  <!-- <gazebo>
-    <plugin filename="libgazebo_ros2_control.so" name="gazebo_ros2_control">
+  </ros2_control>
+  <gazebo>
+    <plugin name="ign_ros2_control::IgnitionROS2ControlPlugin"
+      filename="ign_ros2_control-system">
       <parameters>$(find pendubot_description)/config/effort_control.yaml</parameters>
     </plugin>
-  </gazebo> -->
-<gazebo>
-    <plugin name="ign_ros2_control::IgnitionROS2ControlPlugin"
-        filename="ign_ros2_control-system">
-        <parameters>$(find pendubot_description)/config/effort_control.yaml</parameters>
-    </plugin>
-</gazebo>
+  </gazebo>
 </robot>
